File: cbEval.Stripboard.kicad_pcb (KiCad board)
At the start: 2 copper layers, 35 x 109 mm, 25 parts, among them J1 Bergstik-II_3, J10 Socket.Hor.2x5.6-5535512-4, J11 Bergstik-II_3, J12 Bergstik-II_3, J13 Bergstik-II_6, J14 Bergstik-II_8, J15 Bergstik-II_6, J2 Bergstik-II_6, J3 Keystone.4918, J4 Keystone.4918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

Commit message: kleinere Korrekturen
Parts:
- added H2: Stripfield-4x4, BTech.PCB:Stripfield-4x4, F.Cu at (149.9, 119.4)
- added H3: Stripfield-4x4, BTech.PCB:Stripfield-4x4, F.Cu at (139.7, 119.4)
- added H4: Stripfield-4x4, BTech.PCB:Stripfield-4x4, F.Cu at (149.9, 109.2)
- added H5: Stripfield-4x4, BTech.PCB:Stripfield-4x4, F.Cu at (139.7, 109.2)
- added H6: Stripfield-4x4, BTech.PCB:Stripfield-4x4, F.Cu at (149.9, 99.1)
- added H7: Stripfield-4x4, BTech.PCB:Stripfield-4x4, F.Cu at (139.7, 99.1)
- added H8: Stripfield-4x4, BTech.PCB:Stripfield-4x4, F.Cu at (149.9, 88.9)
- added H9: Stripfield-4x4, BTech.PCB:Stripfield-4x4, F.Cu at (139.7, 88.9)
- moved J14 1.27 mm to (132.1, 126.4)
- moved J11 0.63 mm to (154.9, 126.4)
