File: cbEval.Stripboard.kicad_sch (KiCad schematic)
At the start: 25 parts, among them J1 Bergstik-II_3, J10 Socket.Hor.2x5.6-5535512-4, J11 Bergstik-II_3, J12 Bergstik-II_3, J13 Bergstik-II_6, J14 Bergstik-II_8, J15 Bergstik-II_6, J2 Bergstik-II_6, J3 Keystone.4918, J4 Keystone.4918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

Commit message: kleinere Korrekturen
Parts:
- added H2, H3, H4, H5, H6, H7, H8, H9: Stripfield-4x4, BTech.PCB:Stripfield-4x4, symbol PCB:Stripfield-4x4
Changed lines of the file:
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@@
     (pin "6")
+  )
+  (symbol (lib_id "PCB:Stripfield-4x4") (at 83.82 25.4 0) (unit 1)
+    (in_bom yes) (on_board yes)
+    (property "Reference" "H2" (id 0) (at 83.82 15.24 0))
+    (property "Value" "Stripfield-4x4" (id 1) (at 83.82 17.78 0))
+    (property "Footprint" "BTech.PCB:Stripfield-4x4" (id 2) (at 83.82 12.7 0)
+      (effects (font (size 1.27 1.27)) hide)
+    )
+    (property "Datasheet" "" (id 3) (at 83.82 25.4 0)
+      (effects (font (size 1.27 1.27)) hide)
+    )
+  )
+  (symbol (lib_id "PCB:Stripfield-4x4") (at 83.82 43.18 0) (unit 1)
+    (in_bom yes) (on_board yes)
+    (property "Reference" "H3" (id 0) (at 83.82 33.02 0))
+    (property "Value" "Stripfield-4x4" (id 1) (at 83.82 35.56 0))
+    (property "Footprint" "BTech.PCB:Stripfield-4x4" (id 2) (at 83.82 30.48 0)
+      (effects (font (size 1.27 1.27)) hide)
+    )
+    (property "Datasheet" "" (id 3) (at 83.82 43.18 0)
+      (effects (font (size 1.27 1.27)) hide)
+    )
+  )
+  (symbol (lib_id "PCB:Stripfield-4x4") (at 99.06 25.4 0) (unit 1)
+    (in_bom yes) (on_board yes)
+    (property "Reference" "H4" (id 0) (at 99.06 15.24 0))
+    (property "Value" "Stripfield-4x4" (id 1) (at 99.06 17.78 0))
+    (property "Footprint" "BTech.PCB:Stripfield-4x4" (id 2) (at 99.06 12.7 0)
+      (effects (font (size 1.27 1.27)) hide)
+    )
+    (property "Datasheet" "" (id 3) (at 99.06 25.4 0)
+      (effects (font (size 1.27 1.27)) hide)
+    )
+  )
+  (symbol (lib_id "PCB:Stripfield-4x4") (at 99.06 43.18 0) (unit 1)
+    (in_bom yes) (on_board yes)
+    (property "Reference" "H5" (id 0) (at 99.06 33.02 0))
+    (property "Value" "Stripfield-4x4" (id 1) (at 99.06 35.56 0))
+    (property "Footprint" "BTech.PCB:Stripfield-4x4" (id 2) (at 99.06 30.48 0)
+      (effects (font (size 1.27 1.27)) hide)
+    )
+    (property "Datasheet" "" (id 3) (at 99.06 43.18 0)
+      (effects (font (size 1.27 1.27)) hide)
+    )
+  )
+  (symbol (lib_id "PCB:Stripfield-4x4") (at 114.3 25.4 0) (unit 1)
+    (in_bom yes) (on_board yes)
+    (property "Reference" "H6" (id 0) (at 114.3 15.24 0))
+    (property "Value" "Stripfield-4x4" (id 1) (at 114.3 17.78 0))
+    (property "Footprint" "BTech.PCB:Stripfield-4x4" (id 2) (at 114.3 12.7 0)
+      (effects (font (size 1.27 1.27)) hide)
+    )
+    (property "Datasheet" "" (id 3) (at 114.3 25.4 0)
+      (effects (font (size 1.27 1.27)) hide)
+    )
+  )
+  (symbol (lib_id "PCB:Stripfield-4x4") (at 114.3 43.18 0) (unit 1)
+    (in_bom yes) (on_board yes)
+    (property "Reference" "H7" (id 0) (at 114.3 33.02 0))
+    (property "Value" "Stripfield-4x4" (id 1) (at 114.3 35.56 0))
+    (property "Footprint" "BTech.PCB:Stripfield-4x4" (id 2) (at 114.3 30.48 0)
+      (effects (font (size 1.27 1.27)) hide)
+    )
+    (property "Datasheet" "" (id 3) (at 114.3 43.18 0)
+      (effects (font (size 1.27 1.27)) hide)
+    )
+  )
+  (symbol (lib_id "PCB:Stripfield-4x4") (at 129.54 25.4 0) (unit 1)
+    (in_bom yes) (on_board yes)
+    (property "Reference" "H8" (id 0) (at 129.54 15.24 0))
+    (property "Value" "Stripfield-4x4" (id 1) (at 129.54 17.78 0))
+    (property "Footprint" "BTech.PCB:Stripfield-4x4" (id 2) (at 129.54 12.7 0)
+      (effects (font (size 1.27 1.27)) hide)
+    )
+    (property "Datasheet" "" (id 3) (at 129.54 25.4 0)
+      (effects (font (size 1.27 1.27)) hide)
+    )
+  )
+  (symbol (lib_id "PCB:Stripfield-4x4") (at 129.54 43.18 0) (unit 1)
+    (in_bom yes) (on_board yes)
+    (property "Reference" "H9" (id 0) (at 129.54 33.02 0))
+    (property "Value" "Stripfield-4x4" (id 1) (at 129.54 35.56 0))
+    (property "Footprint" "BTech.PCB:Stripfield-4x4" (id 2) (at 129.54 30.48 0)
+      (effects (font (size 1.27 1.27)) hide)
+    )
+    (property "Datasheet" "" (id 3) (at 129.54 43.18 0)
+      (effects (font (size 1.27 1.27)) hide)
+    )
   )
   (symbol (lib_id "J.PinHeader:Bergstik-II_6") (at 35.56 175.26 0) (mirror y) (unit 1)
@@
       (reference "H1") (unit 1) (value "CIME.E.BE3500S.1x") (footprint "BTech.Housing:Camdenboss.CIME.E.BE3500S.1x")
     )
+    (path "/471ffadc-066e-4d7e-a5b6-ed8f078884cc"
+      (reference "H2") (unit 1) (value "Stripfield-4x4") (footprint "BTech.PCB:Stripfield-4x4")
+    )
+    (path "/f80236f0-de43-4275-850e-32368bcb8c5d"
+      (reference "H3") (unit 1) (value "Stripfield-4x4") (footprint "BTech.PCB:Stripfield-4x4")
+    )
+    (path "/beb48bc0-bb73-4736-b585-f666e49f5901"
+      (reference "H4") (unit 1) (value "Stripfield-4x4") (footprint "BTech.PCB:Stripfield-4x4")
+    )
+    (path "/dc45d19a-5d55-454e-8c51-17387bdf52a0"
+      (reference "H5") (unit 1) (value "Stripfield-4x4") (footprint "BTech.PCB:Stripfield-4x4")
+    )
+    (path "/af335771-b969-45ff-82ec-4b913372caa1"
+      (reference "H6") (unit 1) (value "Stripfield-4x4") (footprint "BTech.PCB:Stripfield-4x4")
+    )
+    (path "/1f993b2f-9d5a-4457-9fbb-14f0f1a712e8"
+      (reference "H7") (unit 1) (value "Stripfield-4x4") (footprint "BTech.PCB:Stripfield-4x4")
+    )
+    (path "/c9b042bc-fe5d-4b69-927f-d62c32a9b41d"
+      (reference "H8") (unit 1) (value "Stripfield-4x4") (footprint "BTech.PCB:Stripfield-4x4")
+    )
+    (path "/a92dcb5a-85d3-416f-8dba-5246b3e17d01"
+      (reference "H9") (unit 1) (value "Stripfield-4x4") (footprint "BTech.PCB:Stripfield-4x4")
+    )
     (path "/4834df8a-150d-455f-b45b-f7736ed80148"
